File: hardware/RPi_Hat.kicad_pcb (KiCad board)
At the start: 2 copper layers, 65 x 56.5 mm, 5 parts, among them J1 RPi_GPIO

Commit message: Semi finished pcb
Parts:
- added C1: 2n, Capacitors_SMD:C_0805_HandSoldering, B.Cu at (67.2, 71.8)
- added C11: 2n, Capacitors_SMD:C_0805_HandSoldering, B.Cu at (116.4, 73.8)
- added C12: CP, Capacitors_THT:CP_Radial_D8.0mm_P3.50mm, F.Cu at (101.0, 85.6)
- added C13: CP, Capacitors_THT:CP_Radial_D8.0mm_P3.50mm, F.Cu at (110.0, 85.6)
- added C14: CP, Capacitors_THT:CP_Radial_D8.0mm_P3.50mm, F.Cu at (119.0, 85.6)
- added C2: 2n, Capacitors_SMD:C_0805_HandSoldering, B.Cu at (73.8, 74.2)
- added C3: 2n, Capacitors_SMD:C_0805_HandSoldering, B.Cu at (73.8, 76.2)
- added C4: 10n, Capacitors_SMD:C_0805_HandSoldering, F.Cu at (79.0, 78.0)
- added C5: 10n, Capacitors_SMD:C_0805_HandSoldering, F.Cu at (84.6, 77.0)
- added C6: 2n, Capacitors_SMD:C_0805_HandSoldering, F.Cu at (72.0, 66.0)
- added C7: 2n, Capacitors_SMD:C_0805_HandSoldering, B.Cu at (105.8, 71.6)
- added C8: C, Capacitors_SMD:C_0805_HandSoldering, F.Cu at (90.6, 58.4)
- added C9: 2n, Capacitors_SMD:C_0805_HandSoldering, B.Cu at (80.8, 67.4)
- added D1: DIODESCH, Diodes_SMD:D_SMA_Handsoldering, F.Cu at (86.4, 92.2)
- added D10: DIODESCH, Diodes_SMD:D_SMA_Handsoldering, F.Cu at (86.4, 85.0)
- added D11: LED, Diodes_SMD:D_0805, F.Cu at (126.6, 91.6)
- added D12: LED, Diodes_SMD:D_0805, F.Cu at (126.6, 93.8)
- added D13: ZENER, Diodes_SMD:D_SOD-123F, F.Cu at (111.4, 92.6)
- added D2: DIODESCH, Diodes_SMD:D_SMA_Handsoldering, F.Cu at (76.2, 85.1)
- added D3: DIODESCH, Diodes_SMD:D_SMA_Handsoldering, F.Cu at (75.8, 92.2)
- added D4: ZENER, Diodes_SMD:D_SOD-123F, F.Cu at (81.2, 101.8)
- added D5: ZENER, Diodes_SMD:D_SOD-123F, B.Cu at (75.0, 100.2)
- added D6: ZENER, Diodes_SMD:D_SOD-123F, B.Cu at (74.8, 84.2)
- added D7: ZENER, Diodes_SMD:D_SOD-123F, B.Cu at (74.8, 92.4)
- added D8: DIODESCH, Diodes_SMD:D_SMA_Handsoldering, F.Cu at (76.2, 81.0)
- added D9: ZENER, Diodes_SMD:D_SOD-123F, F.Cu at (125.8, 87.2)
- added IC1: ATTINY1634-S, Housings_SOIC:SO-20_12.8x7.5mm_Pitch1.27mm, F.Cu at (80.8, 63.2)
- added P1: CONN_2, Connectors_Molex:Molex_KK-6410-02_02x2.54mm_Straight, F.Cu at (92.7, 101.6)
- added P2: CONN_2, Connectors_Molex:Molex_KK-6410-02_02x2.54mm_Straight, F.Cu at (67.3, 85.1)
- added P3: CONN_2, Connectors_Molex:Molex_KK-6410-02_02x2.54mm_Straight, F.Cu at (67.3, 92.7)
- added P4: CONN_2, Connectors_Molex:Molex_KK-6410-02_02x2.54mm_Straight, F.Cu at (67.0, 59.5)
- added P5: CONN_2, Connectors_Molex:Molex_KK-6410-02_02x2.54mm_Straight, F.Cu at (113.0, 101.6)
- added P6: Conn_02x03_Odd_Even, extras:Header_2x03, F.Cu at (89.6, 62.6)
- added Q1: DMP3056L-7, TO_SOT_Packages_SMD:SOT-23_Handsoldering, F.Cu at (88.8, 97.0)
- added Q10: BC846BPDW1, TO_SOT_Packages_SMD:SOT-363_SC-70-6_Handsoldering, F.Cu at (67.2, 74.6)
- added Q2: DMP3056L-7, TO_SOT_Packages_SMD:SOT-23_Handsoldering, F.Cu at (83.8, 97.0)
- added Q3: DMP3056L-7, TO_SOT_Packages_SMD:SOT-23_Handsoldering, F.Cu at (76.2, 88.9)
- added Q4: DMP3056L-7, TO_SOT_Packages_SMD:SOT-23_Handsoldering, F.Cu at (76.6, 96.0)
- added Q5: NPN, TO_SOT_Packages_SMD:SOT-23_Handsoldering, B.Cu at (100.2, 68.0)
- added Q6: DMP3056L-7, TO_SOT_Packages_SMD:SOT-23_Handsoldering, F.Cu at (125.2, 81.8)
- added Q7: NPN, TO_SOT_Packages_SMD:SOT-23_Handsoldering, B.Cu at (111.4, 67.8)
- added Q8: DMP3056L-7, TO_SOT_Packages_SMD:SOT-23_Handsoldering, F.Cu at (108.0, 95.0)
- added Q9: NPN, TO_SOT_Packages_SMD:SOT-23_Handsoldering, B.Cu at (111.4, 63.6)
- added R10: 47K, Resistors_SMD:R_0805_HandSoldering, B.Cu at (84.2, 101.6)
- added R11: 47K, Resistors_SMD:R_0805_HandSoldering, B.Cu at (83.8, 83.6)
- added R12: 47K, Resistors_SMD:R_0805_HandSoldering, B.Cu at (83.8, 85.6)
- added R13: 47K, Resistors_SMD:R_0805_HandSoldering, B.Cu at (84.0, 91.8)
- added R14: 47K, Resistors_SMD:R_0805_HandSoldering, B.Cu at (84.0, 93.8)
- added R15: 10K, Resistors_SMD:R_0805_HandSoldering, F.Cu at (72.0, 60.8)
- added R16: 10K, Resistors_SMD:R_0805_HandSoldering, B.Cu at (105.8, 73.8)
- added R17: 100K, Resistors_SMD:R_0805_HandSoldering, F.Cu at (125.6, 84.8)
- added R18: 220R, Resistors_SMD:R_0805_HandSoldering, F.Cu at (121.8, 91.6)
- added R19: 1K, Resistors_SMD:R_0805_HandSoldering, F.Cu at (67.2, 65.8)
- added R2: 100K, Resistors_SMD:R_0805_HandSoldering, F.Cu at (88.0, 101.8)
- added R20: 1K, Resistors_SMD:R_0805_HandSoldering, B.Cu at (100.4, 73.8)
- added R21: 220R, Resistors_SMD:R_0805_HandSoldering, F.Cu at (121.8, 93.8)
- added R22: 500K, Resistors_SMD:R_0805_HandSoldering, B.Cu at (105.8, 67.0)
- added R23: 100K, Resistors_SMD:R_0805_HandSoldering, F.Cu at (113.8, 92.6)
- added R24: 500K, Resistors_SMD:R_0805_HandSoldering, B.Cu at (105.8, 62.6)
- added R25: 5m, Resistors_SMD:R_2010_HandSoldering, F.Cu at (86.6, 88.6)
- added R26: R, Resistors_SMD:R_0805_HandSoldering, F.Cu at (67.2, 71.8)
- added R27: 500K, Resistors_SMD:R_0805_HandSoldering, F.Cu at (67.2, 77.2)
- added R3: 10K, Resistors_SMD:R_0805_HandSoldering, F.Cu at (73.8, 70.2)
- added R30: 500K, Resistors_SMD:R_0805_HandSoldering, F.Cu at (67.2, 67.8)
- added R31: 10K, Resistors_SMD:R_0805_HandSoldering, B.Cu at (111.2, 71.4)
- added R32: 1K, Resistors_SMD:R_0805_HandSoldering, B.Cu at (111.2, 73.8)
- added R4: 10K, Resistors_SMD:R_0805_HandSoldering, F.Cu at (73.8, 74.2)
- added R5: R, Resistors_SMD:R_0805_HandSoldering, F.Cu at (67.2, 69.8)
- added R6: 1K, Resistors_SMD:R_0805_HandSoldering, F.Cu at (73.8, 72.2)
- added R7: 1K, Resistors_SMD:R_0805_HandSoldering, F.Cu at (73.8, 76.2)
- added R8: 500K, Resistors_SMD:R_0805_HandSoldering, B.Cu at (105.8, 69.2)
- added R9: 47K, Resistors_SMD:R_0805_HandSoldering, B.Cu at (84.2, 99.2)
- added RV1: POT, Potentiometers:Potentiometer_Trimmer_Bourns_PV36W, F.Cu at (90.8, 79.8)
- added S1: BUCKCNV, extras:BUCK, F.Cu at (100.8, 70.2)
- added S2: BUCKCNV, extras:BUCK, F.Cu at (118.0, 70.2)
- added S3: BUCKCNV-CC, Connectors_Molex:Molex_KK-6410-04_04x2.54mm_Straight, F.Cu at (100.3, 101.6)
- added U1: DMMT5401, TO_SOT_Packages_SMD:SOT-23-6_Handsoldering, B.Cu at (79.2, 100.4)
- added U2: DMMT5401, TO_SOT_Packages_SMD:SOT-23-6_Handsoldering, B.Cu at (78.8, 84.6)
- added U3: DMMT5401, TO_SOT_Packages_SMD:SOT-23-6_Handsoldering, B.Cu at (78.8, 92.8)
- added U4: XC6216, TO_SOT_Packages_SMD:SOT-23-5_HandSoldering, F.Cu at (79.2, 74.8)
- added U5: MAX44284, TO_SOT_Packages_SMD:SOT-23-6_Handsoldering, F.Cu at (84.6, 80.0)
Connections:
- J1 pad 14: Net-(J1-Pad14) -> DGND
- J1 pad 2: Net-(J1-Pad2) -> +5V
- J1 pad 20: Net-(J1-Pad14) -> DGND
- J1 pad 25: Net-(J1-Pad25) -> DGND
- J1 pad 3: Net-(J1-Pad3) -> /MOSI
- J1 pad 30: Net-(J1-Pad30) -> DGND
- J1 pad 32: Net-(J1-Pad24) -> Net-(J1-Pad32)
- J1 pad 34: Net-(J1-Pad34) -> DGND
- J1 pad 39: Net-(J1-Pad39) -> DGND
- J1 pad 4: Net-(J1-Pad4) -> +5V
- J1 pad 5: Net-(J1-Pad5) -> /SCK
- J1 pad 6: Net-(J1-Pad6) -> DGND
- J1 pad 9: Net-(J1-Pad9) -> DGND
Routing:
- net +5V: track 0.00 -> 133.9 mm
- net /BATT: track 0.00 -> 95.3 mm
- net /LED_GREEN: track 0.00 -> 80.8 mm, vias 0 -> 2
- net /LED_RED: track 0.00 -> 79.4 mm, vias 0 -> 2
- net Net-(P5-Pad1): track 0.00 -> 74.6 mm, vias 0 -> 19
- net /PBUS_IN: track 0.00 -> 65.4 mm, vias 0 -> 3
- net Net-(D4-Pad2): track 0.00 -> 64.3 mm, vias 0 -> 3
- net /S_AUXOUT: track 0.00 -> 54.8 mm, vias 0 -> 3
- net /EN_CURRMON: track 0.00 -> 46.0 mm, vias 0 -> 4
- net Net-(D13-Pad2): track 0.00 -> 44.0 mm, vias 0 -> 1
- net VCC: track 0.00 -> 42.0 mm, vias 0 -> 3
- net /AUX2: track 0.00 -> 36.7 mm, vias 0 -> 3
- net DGND: track 0.00 -> 36.1 mm, vias 0 -> 12
- net /EN_AUXOUT: track 0.00 -> 33.9 mm, vias 0 -> 3
- net /S_PBUS: track 0.00 -> 31.6 mm, vias 0 -> 1
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- added copper zone on F.Cu, net +5V
- added copper zone on F.Cu, net /AUX1
- added copper zone on F.Cu, net /AUX2
- added copper zone on F.Cu, net /PBUS
- added copper zone on F.Cu, net /PBUS_IN
- added copper zone on B.Cu, net DGND
- added copper zone on F.Cu, net Net-(D1-Pad2)
- added copper zone on B.Cu, net Net-(P5-Pad1)
- added copper zone on F.Cu, net Net-(P5-Pad1)
Other:
- outline, holes or cut-outs redrawn
- board text added: "5V"
- board text added: "AUX1"
- board text added: "AUX2"
- board text added: "AUXOUT"
- board text added: "BATT"
- board text added: "CHGPSU"

Commit message: First PCB version
Routing:
- net Net-(D4-Pad2): track 64.3 -> 81.0 mm
- net /PBUS: track 23.0 -> 27.4 mm
- net +5V: track 133.9 -> 137.1 mm
- net /AUX2: track 36.7 -> 35.4 mm
- net /LED_GREEN: track 80.8 -> 79.7 mm
- net Net-(P5-Pad1): track 74.6 -> 75.5 mm
- net /EN_AUXOUT: track 33.9 -> 33.2 mm
- added copper zone on F.Cu, net /BATT
- added copper zone on F.Cu, net Net-(Q8-Pad3)
Other:
- board text added: "B52/BUSHFIRE REV1/2017/11 E/OVERTON"
